Commit message: 完成关节控制\麦克纳姆轮控制器的配置

File: src/kai01_description/ros2_control/kai01.ros2_control.xacro (robot description, xacro)
@@ -5,4 +5,5 @@
       <hardware>
         <plugin>mock_components/GenericSystem</plugin> <!-- 使用虚拟组件快速测试 -->
+        <param name="calculate_dynamics">true</param>
       </hardware>
       <joint name="${prefix}arm_joint1">  <!-- 机械臂第1旋转关节 -->
@@ -60,13 +61,4 @@
         </state_interface>
       </joint>
-      <joint name="${prefix}arm_joint6">   <!-- 机械臂第6旋转关节 -->
-        <command_interface name="position">
-          <param name="min">-2.09</param>
-          <param name="max">2.09</param>
-        </command_interface>
-        <state_interface name="position">
-          <param name="initial_value">0.0</param>
-        </state_interface>
-      </joint>
       <joint name="${prefix}wheel_left_front_joint">   <!-- 左前轮 -->
         <command_interface name="velocity">
@@ -77,4 +69,5 @@
           <param name="initial_value">0.0</param>
         </state_interface>
+        <state_interface name="position"/>
       </joint>
       <joint name="${prefix}wheel_left_back_joint">   <!-- 左后轮 -->
@@ -86,4 +79,5 @@
           <param name="initial_value">0.0</param>
         </state_interface>
+        <state_interface name="position"/>
       </joint>
       <joint name="${prefix}wheel_right_front_joint">   <!-- 右前轮 -->
@@ -95,4 +89,5 @@
           <param name="initial_value">0.0</param>
         </state_interface>
+        <state_interface name="position"/>
       </joint>
       <joint name="${prefix}wheel_right_back_joint">   <!-- 右后轮 -->
@@ -104,13 +99,6 @@
           <param name="initial_value">0.0</param>
         </state_interface>
+        <state_interface name="position"/>
       </joint>
-      <sensor name="${prefix}imu">   <!-- imu -->
-        <state_interface name="accel_x"/>  <!-- x轴加速度 -->
-        <state_interface name="accel_y"/>  <!-- y轴加速度 -->
-        <state_interface name="accel_y"/>  <!-- z轴加速度-->
-        <state_interface name="gyro_x"/>  <!--  x轴角速度 -->
-        <state_interface name="gyro_y"/>  <!--  y轴角速度 -->
-        <state_interface name="gyro_z"/>  <!--  z轴角速度-->
-      </sensor>
     </ros2_control>
   </xacro:macro>

Commit message: 增加moveit_config包

File: src/kai01_description/ros2_control/kai01.ros2_control.xacro (robot description, xacro)
@@ -2,104 +2,135 @@
 <robot xmlns:xacro="http://www.ros.org/wiki/xacro">
   <xacro:macro name="kai01_interface" params="name prefix">
-    <ros2_control name="${name}" type="system">
-      <hardware>
-        <plugin>mock_components/GenericSystem</plugin> <!-- 使用虚拟组件快速测试 -->
-        <param name="calculate_dynamics">true</param>
-      </hardware>
-      <joint name="${prefix}arm_joint1">  <!-- 机械臂第1旋转关节 -->
-        <command_interface name="position">
-          <param name="min">-2.09</param>
-          <param name="max">2.09</param>
-        </command_interface>
-        <state_interface name="position">
-          <param name="initial_value">0.0</param>
-        </state_interface>
-      </joint>
-      <joint name="${prefix}arm_joint2">   <!-- 机械臂第2旋转关节 -->
-        <command_interface name="position">
-          <param name="min">-2.09</param>
-          <param name="max">2.09</param>
-        </command_interface>
-        <state_interface name="position">
-          <param name="initial_value">0.0</param>
-        </state_interface>
-      </joint>
-      <joint name="${prefix}arm_joint3">   <!-- 机械臂第3旋转关节 -->
-        <command_interface name="position">
-          <param name="min">-2.09</param>
-          <param name="max">2.09</param>
-        </command_interface>
-        <state_interface name="position">
-          <param name="initial_value">0.0</param>
-        </state_interface>
-      </joint>
-      <joint name="${prefix}arm_joint4">   <!-- 机械臂第4旋转关节 -->
-        <command_interface name="position">
-          <param name="min">-2.09</param>
-          <param name="max">2.09</param>
-        </command_interface>
-        <state_interface name="position">
-          <param name="initial_value">0.0</param>
-        </state_interface>
-      </joint>
-      <joint name="${prefix}arm_joint5">   <!-- 机械臂第5旋转关节 -->
-        <command_interface name="position">
-          <param name="min">-2.09</param>
-          <param name="max">2.09</param>
-        </command_interface>
-        <state_interface name="position">
-          <param name="initial_value">0.0</param>
-        </state_interface>
-      </joint>
-      <joint name="${prefix}arm_joint6">   <!-- 机械臂第6旋转关节 -->
-        <command_interface name="position">
-          <param name="min">-2.09</param>
-          <param name="max">2.09</param>
-        </command_interface>
-        <state_interface name="position">
-          <param name="initial_value">0.0</param>
-        </state_interface>
-      </joint>
-      <joint name="${prefix}wheel_left_front_joint">   <!-- 左前轮 -->
-        <command_interface name="velocity">
-          <param name="min">-2.0</param>
-          <param name="max">2.0</param>
-        </command_interface>
-        <state_interface name="velocity">
-          <param name="initial_value">0.0</param>
-        </state_interface>
-        <state_interface name="position"/>
-      </joint>
-      <joint name="${prefix}wheel_left_back_joint">   <!-- 左后轮 -->
-        <command_interface name="velocity">
-          <param name="min">-2.0</param>
-          <param name="max">2.0</param>
-        </command_interface>
-        <state_interface name="velocity">
-          <param name="initial_value">0.0</param>
-        </state_interface>
-        <state_interface name="position"/>
-      </joint>
-      <joint name="${prefix}wheel_right_front_joint">   <!-- 右前轮 -->
-        <command_interface name="velocity">
-          <param name="min">-2.0</param>
-          <param name="max">2.0</param>
-        </command_interface>
-        <state_interface name="velocity">
-          <param name="initial_value">0.0</param>
-        </state_interface>
-        <state_interface name="position"/>
-      </joint>
-      <joint name="${prefix}wheel_right_back_joint">   <!-- 右后轮 -->
-        <command_interface name="velocity">
-          <param name="min">-2.0</param>
-          <param name="max">2.0</param>
-        </command_interface>
-        <state_interface name="velocity">
-          <param name="initial_value">0.0</param>
-        </state_interface>
-        <state_interface name="position"/>
-      </joint>
-    </ros2_control>
+  <!-- ========== ros2_control hardware interface ========== -->
+  <ros2_control name="RobotBoardSystem" type="system">
+    <hardware>
+      <plugin>robot_board_hardware/RobotBoardSystemInterface</plugin>
+      <param name="serial_port">/dev/ttyACM0</param>
+      <param name="baud_rate">1000000</param>
+    </hardware>
+    <!-- 4 Mecanum wheel motors: velocity command/state -->
+    <!-- Physical wiring: motor1=FL(左前), motor2=RL(左后), motor3=FR(右前), motor4=RR(右后) -->
+    <!-- Right-side motors (3,4) are mounted reversed; negate is applied in robot_board_hardware -->
+    <joint name="wheel_left_front_joint">
+      <command_interface name="velocity"/>
+      <state_interface name="position"/>
+      <state_interface name="velocity"/>
+      <param name="motor_id">1</param>
+    </joint>
+    <joint name="wheel_left_back_joint">
+      <command_interface name="velocity"/>
+      <state_interface name="position"/>
+      <state_interface name="velocity"/>
+      <param name="motor_id">2</param>
+    </joint>
+    <joint name="wheel_right_front_joint">
+      <command_interface name="velocity"/>
+      <state_interface name="position"/>
+      <state_interface name="velocity"/>
+      <param name="motor_id">3</param>
+    </joint>
+    <joint name="wheel_right_back_joint">
+      <command_interface name="velocity"/>
+      <state_interface name="position"/>
+      <state_interface name="velocity"/>
+      <param name="motor_id">4</param>
+    </joint>
+    <joint name="arm_joint1">
+      <command_interface name="position"/>
+      <state_interface name="position"/>
+      <param name="servo_id">1</param>
+      <param name="zero">498</param>
+      <param name="init">0.0</param>
+      <param name="min">1000</param>
+      <param name="max">0</param>
+      <param name="servo_duration">1200</param>
+    </joint>
+    <joint name="arm_joint2">
+      <command_interface name="position"/>
+      <state_interface name="position"/>
+      <param name="servo_id">2</param>
+      <param name="zero">495</param>
+      <param name="init">-0.9</param>
+      <param name="min">1000</param>
+      <param name="max">0</param>
+      <param name="servo_duration">1200</param>
+    </joint>
+    <joint name="arm_joint3">
+      <command_interface name="position"/>
+      <state_interface name="position"/>
+      <param name="servo_id">3</param>
+      <param name="zero">470</param>
+      <param name="init">1.57</param>
+      <param name="min">1000</param>
+      <param name="max">0</param>
+      <param name="servo_duration">1200</param>
+    </joint>
+    <joint name="arm_joint4">
+      <command_interface name="position"/>
+      <state_interface name="position"/>
+      <param name="servo_id">4</param>
+      <param name="zero">511</param>
+      <param name="init">1.57</param>
+      <param name="min">1000</param>
+      <param name="max">0</param>
+      <param name="servo_duration">1200</param>
+    </joint>
+    <joint name="arm_joint5">
+      <command_interface name="position"/>
+      <state_interface name="position"/>
+      <param name="servo_id">5</param>
+      <param name="zero">504</param>
+      <param name="init">0.0</param>
+      <param name="min">1000</param>
+      <param name="max">0</param>
+      <param name="servo_duration">1200</param>
+    </joint>
+    <joint name="arm_joint6">
+      <command_interface name="position"/>
+      <state_interface name="position"/>
+      <param name="servo_id">10</param>
+      <param name="zero">591</param>
+      <param name="init">0.0</param>
+      <param name="min">1000</param>
+      <param name="max">0</param>
+      <param name="servo_duration">1200</param>
+    </joint>
+    <!-- IMU sensor -->
+    <sensor name="imu_sensor">
+      <state_interface name="orientation.x"/>
+      <state_interface name="orientation.y"/>
+      <state_interface name="orientation.z"/>
+      <state_interface name="orientation.w"/>
+      <state_interface name="angular_velocity.x"/>
+      <state_interface name="angular_velocity.y"/>
+      <state_interface name="angular_velocity.z"/>
+      <state_interface name="linear_acceleration.x"/>
+      <state_interface name="linear_acceleration.y"/>
+      <state_interface name="linear_acceleration.z"/>
+    </sensor>
+    <!-- Battery voltage sensor -->
+    <sensor name="battery_sensor">
+      <state_interface name="voltage"/>
+    </sensor>
+    <!-- Button sensor -->
+    <sensor name="button_sensor">
+      <state_interface name="button1_state"/>
+      <state_interface name="button2_state"/>
+    </sensor>
+    <!-- LED GPIO -->
+    <gpio name="led">
+      <command_interface name="on_time"/>
+      <command_interface name="off_time"/>
+      <command_interface name="repeat"/>
+      <command_interface name="led_id"/>
+    </gpio>
+    <!-- Buzzer GPIO -->
+    <gpio name="buzzer">
+      <command_interface name="frequency"/>
+      <command_interface name="on_time"/>
+      <command_interface name="off_time"/>
+      <command_interface name="repeat"/>
+    </gpio>
+  </ros2_control>
   </xacro:macro>
 </robot>

File: src/kai01_description/urdf/arm_moveit.urdf.xacro (robot description, xacro)
@@ -2,4 +2,26 @@
 <robot name="arm" xmlns:xacro="http://ros.org/wiki/xacro">
   <xacro:property name="M_PI"   value="3.1415926535897931"/>
+  <link
+    name="base_link"> <!-- 移动底盘底座 -->
+  </link>
+<!-- 机械臂底座连接关节 -->
+  <joint
+    name="arm_joint1"
+    type="revolute">
+    <origin
+      xyz="0.0251328065010765 0 0.0774026880954513"
+      rpy="0 0 0" />
+    <parent
+      link="base_link" />
+    <child
+      link="arm_base_link" />
+    <axis
+      xyz="0 0 -1" />
+    <limit
+      lower="-2.09"
+      upper="2.09"
+      effort="1000"
+      velocity="10" />
+  </joint>
   <link
     name="arm_base_link"> <!-- 机械臂底座 -->
@@ -26,5 +48,4 @@
           filename="package://kai01_description/meshes/arm/arm_base_link.STL" />
       </geometry>
-      <material name="green"/>
     </visual>
     <collision>
@@ -129,5 +150,4 @@
           filename="package://kai01_description/meshes/arm/Link_1.STL" />
       </geometry>
-      <material name="green"/>
     </visual>
     <collision>
@@ -183,5 +203,4 @@
           filename="package://kai01_description/meshes/arm/Link_2.STL" />
       </geometry>
-      <material name="green"/>
     </visual>
     <collision>
@@ -237,5 +256,4 @@
           filename="package://kai01_description/meshes/arm/Link_3.STL" />
       </geometry>
-      <material name="green"/>
     </visual>
     <collision>
@@ -352,18 +370,4 @@
     </collision>
   </link>
-  <link name="gripper" /> <!-- 夹爪中心点（虚拟） -->
-  <joint
-    name="gripper_to_tcp"
-    type="fixed">
-    <origin
-      xyz="0 0 0.065"
-      rpy="0 0 0" />
-    <parent
-      link="coupling" />
-    <child
-      link="gripper" />
-    <axis
-      xyz="0 0 0" />
-  </joint>
   <joint
     name="gripper_joint"

File: src/kai01_description/urdf/kai01.urdf.xacro (robot description, xacro)
@@ -9,7 +9,5 @@
   <!-- 硬件接口 -->
   <xacro:include filename="$(find kai01_description)/ros2_control/kai01.ros2_control.xacro"/><!-- 硬件接口描述 -->
-  <xacro:kai01_interface
-    name= "KAI01_INTERFACE"
-    prefix="$(arg prefix)" />
+  <xacro:kai01_interface name="RobotBoardSystem" prefix=""/>
 <!-- 机械臂底座连接关节 -->
   <joint

File: src/robot_bringup/urdf/robot.urdf.xacro (robot description, xacro)
@@ -67,4 +67,6 @@
     </hardware>
     <!-- 4 Mecanum wheel motors: velocity command/state -->
+    <!-- Physical wiring: motor1=FL(左前), motor2=RL(左后), motor3=FR(右前), motor4=RR(右后) -->
+    <!-- Right-side motors (3,4) are mounted reversed; negate is applied in robot_board_hardware -->
     <joint name="front_left_wheel_joint">
       <command_interface name="velocity"/>
@@ -72,15 +74,15 @@
       <param name="motor_id">1</param>
     </joint>
-    <joint name="front_right_wheel_joint">
+    <joint name="rear_left_wheel_joint">
       <command_interface name="velocity"/>
       <state_interface name="velocity"/>
       <param name="motor_id">2</param>
     </joint>
-    <joint name="rear_right_wheel_joint">
+    <joint name="front_right_wheel_joint">
       <command_interface name="velocity"/>
       <state_interface name="velocity"/>
       <param name="motor_id">3</param>
     </joint>
-    <joint name="rear_left_wheel_joint">
+    <joint name="rear_right_wheel_joint">
       <command_interface name="velocity"/>
       <state_interface name="velocity"/>
@@ -88,8 +90,16 @@
     </joint>
     <!-- 6 Bus servos for robot arm: position command/state (radians) -->
+    <!-- Parameters: servo_id, zero (pulse at 0 rad), init (initial angle in rad), min/max in pulse width, servo_duration in ms -->
+    <!-- When min > max, the joint is flipped (reversed direction) -->
+    <!-- servo_duration: movement duration in ms (0=fastest, larger=slower) -->
     <joint name="arm_joint_1">
       <command_interface name="position"/>
       <state_interface name="position"/>
       <param name="servo_id">1</param>
+      <param name="zero">498</param>
+      <param name="init">0.0</param>
+      <param name="min">1000</param>
+      <param name="max">0</param>
+      <param name="servo_duration">2000</param>
     </joint>
     <joint name="arm_joint_2">
@@ -97,4 +107,9 @@
       <state_interface name="position"/>
       <param name="servo_id">2</param>
+      <param name="zero">495</param>
+      <param name="init">-0.9</param>
+      <param name="min">1000</param>
+      <param name="max">0</param>
+      <param name="servo_duration">2000</param>
     </joint>
     <joint name="arm_joint_3">
@@ -102,4 +117,9 @@
       <state_interface name="position"/>
       <param name="servo_id">3</param>
+      <param name="zero">470</param>
+      <param name="init">1.57</param>
+      <param name="min">1000</param>
+      <param name="max">0</param>
+      <param name="servo_duration">2000</param>
     </joint>
     <joint name="arm_joint_4">
@@ -107,4 +127,9 @@
       <state_interface name="position"/>
       <param name="servo_id">4</param>
+      <param name="zero">511</param>
+      <param name="init">1.57</param>
+      <param name="min">1000</param>
+      <param name="max">0</param>
+      <param name="servo_duration">2000</param>
     </joint>
     <joint name="arm_joint_5">
@@ -112,9 +137,19 @@
       <state_interface name="position"/>
       <param name="servo_id">5</param>
+      <param name="zero">504</param>
+      <param name="init">0.0</param>
+      <param name="min">1000</param>
+      <param name="max">0</param>
+      <param name="servo_duration">2000</param>
     </joint>
     <joint name="arm_joint_6">
       <command_interface name="position"/>
       <state_interface name="position"/>
-      <param name="servo_id">6</param>
+      <param name="servo_id">10</param>
+      <param name="zero">591</param>
+      <param name="init">0.0</param>
+      <param name="min">1000</param>
+      <param name="max">0</param>
+      <param name="servo_duration">2000</param>
     </joint>
     <!-- IMU sensor -->

Commit message: 6.20备份

File: src/kai01_description/ros2_control/kai01.ros2_control.xacro (robot description, xacro)
@@ -39,4 +39,5 @@
       <command_interface name="position"/>
       <state_interface name="position"/>
+      <state_interface name="velocity"/>
       <param name="servo_id">1</param>
       <param name="zero">498</param>
@@ -49,4 +50,5 @@
       <command_interface name="position"/>
       <state_interface name="position"/>
+      <state_interface name="velocity"/>
       <param name="servo_id">2</param>
       <param name="zero">495</param>
@@ -59,4 +61,5 @@
       <command_interface name="position"/>
       <state_interface name="position"/>
+      <state_interface name="velocity"/>
       <param name="servo_id">3</param>
       <param name="zero">470</param>
@@ -69,4 +72,5 @@
       <command_interface name="position"/>
       <state_interface name="position"/>
+      <state_interface name="velocity"/>
       <param name="servo_id">4</param>
       <param name="zero">511</param>
@@ -79,4 +83,5 @@
       <command_interface name="position"/>
       <state_interface name="position"/>
+      <state_interface name="velocity"/>
       <param name="servo_id">5</param>
       <param name="zero">504</param>
@@ -89,7 +94,8 @@
       <command_interface name="position"/>
       <state_interface name="position"/>
+      <state_interface name="velocity"/>
       <param name="servo_id">10</param>
       <param name="zero">591</param>
-      <param name="init">0.0</param>
+      <param name="init">1.2</param>
       <param name="min">1000</param>
       <param name="max">0</param>

File: src/kai01_description/urdf/arm.urdf.xacro (robot description, xacro)
@@ -352,18 +352,4 @@
     </collision>
   </link>
-  <link name="gripper" /> <!-- 夹爪中心点（虚拟） -->
-  <joint
-    name="gripper_to_tcp"
-    type="fixed">
-    <origin
-      xyz="0 0 0.065"
-      rpy="0 0 0" />
-    <parent
-      link="coupling" />
-    <child
-      link="gripper" />
-    <axis
-      xyz="0 0 0" />
-  </joint>
   <joint
     name="gripper_joint"
@@ -811,5 +797,5 @@
   </joint>
   <link
-    name="depth_cam_link"> <!-- 深度相机 -->
+    name="camera_link"> <!-- 深度相机 -->
     <inertial>
       <origin
@@ -859,15 +845,7 @@
       link="camera_connect_link" />
     <child
-      link="depth_cam_link" />
+      link="camera_link" />
     <axis
       xyz="0 0 0" />
   </joint>
-  <link name="depth_cam_frame" /> <!-- 虚拟相机坐标系 -->
-  <joint
-    name="depth_cam_joint_sim"
-    type="fixed">
-    <origin xyz="0 0 0" rpy="${-M_PI/2} 0 ${-M_PI/2}" />
-    <parent link="depth_cam_link" />
-    <child link="depth_cam_frame" />
-  </joint>
 </robot>

Commit message: 6.28

File: src/kai01_description/ros2_control/kai01.ros2_control.xacro (robot description, xacro)
@@ -6,5 +6,5 @@
     <hardware>
       <plugin>robot_board_hardware/RobotBoardSystemInterface</plugin>
-      <param name="serial_port">/dev/ttyACM0</param>
+      <param name="serial_port">/dev/robot_board</param>
       <param name="baud_rate">1000000</param>
     </hardware>

File: src/kai01_description/urdf/car_mecanum.urdf.xacro (robot description, xacro)
@@ -13,4 +13,10 @@
     <origin xyz="0.0 0.0 ${0.0965/2 + 0.0678410821576746}" rpy="0 0 0"/>
   </joint>
+  <link name="measure"/><!-- 测量点 -->
+  <joint name="measure_joint" type="fixed">
+    <parent link="base_footprint"/>
+    <child link="measure"/>
+    <origin xyz="0.153 0.0 0.0" rpy="0 0 0"/>
+  </joint>
   <link
     name="base_link"> <!-- 下底盘 -->
