Commit message: 7.9

File: src/kai01_description/urdf/car_mecanum.urdf.xacro (robot description, xacro)
@@ -11,11 +11,11 @@
     <parent link="base_footprint"/>
     <child link="base_link"/>
-    <origin xyz="0.0 0.0 ${0.0965/2 + 0.0678410821576746}" rpy="0 0 0"/>
+    <origin xyz="0.0 0.0 0.12" rpy="0 0 0"/>
   </joint>
   <link name="measure"/><!-- 测量点 -->
   <joint name="measure_joint" type="fixed">
-    <parent link="base_footprint"/>
-    <child link="measure"/>
-    <origin xyz="0.153 0.0 0.0" rpy="0 0 0"/>
+    <parent link="measure"/>
+    <child link="base_footprint"/>
+    <origin xyz="-0.153 0.0 0.0" rpy="0 0 0"/>
   </joint>
   <link
